Commit message: adjusted camera and observation pose angles

File: src/realsense2_description-master/urdf/_d435.urdf.xacro (robot description, xacro)
@@ -33,5 +33,5 @@
     <!-- camera body, with origin at bottom screw mount -->
     <joint name="${name}_joint" type="fixed">
-      <origin xyz="0 ${d435_cam_height/2 + 0.02} 0" rpy="-${M_PI/2} 0 0"/>
+      <origin xyz="0 ${d435_cam_height/2 + 0.02} 0" rpy="-${M_PI/2} 0 0.3"/>
       <parent link="${parent}"/>
       <child link="${name}_bottom_screw_frame" />
