Commit message: from ned_camera to d435 publishing now

File: src/niryo_robot_description/urdf/ned/niryo_ned_gripper1_n_camera.urdf.xacro (robot description, xacro)
@@ -1,5 +1,5 @@
 <?xml version="1.0"?>
 <robot xmlns:xacro="http://www.ros.org/wiki/xacro" name="niryo_ned">
-    <xacro:include filename="$(find niryo_robot_description)/urdf/ned/niryo_ned_camera.urdf.xacro"/>
+    <xacro:include filename="$(find realsense2_description)/urdf/test_d435_camera.urdf.xacro"/>
     <!-- gazebo joint state publisher for all joints. Necessary to control mors -->
     <gazebo>

File: src/realsense2_description-master/urdf/_d435.urdf.xacro (robot description, xacro)
@@ -33,5 +33,5 @@
     <!-- camera body, with origin at bottom screw mount -->
     <joint name="${name}_joint" type="fixed">
-      <xacro:insert_block name="origin" />
+      <origin xyz="0 ${d435_cam_height/2 + 0.02} 0" rpy="-${M_PI/2} 0 0"/>
       <parent link="${parent}"/>
       <child link="${name}_bottom_screw_frame" />

File: src/realsense2_description-master/urdf/test_d435_camera.urdf.xacro (robot description, xacro)
@@ -1,7 +1,7 @@
 <?xml version="1.0"?>
 <robot name="realsense2_camera" xmlns:xacro="http://ros.org/wiki/xacro">
+  <xacro:include filename="$(find niryo_robot_description)/urdf/ned/niryo_ned_gazebo.urdf.xacro"/>
   <xacro:include filename="$(find realsense2_description)/urdf/_d435.urdf.xacro" />
-  <link name="base_link" />
-  <xacro:sensor_d435 name="camera" topics_ns="camera" parent="base_link" publish_pointcloud="true">
+  <xacro:sensor_d435 name="camera" topics_ns="camera" parent="wrist_link" publish_pointcloud="true">
     <origin xyz="0 0 0" rpy="0 0 0" />
   </xacro:sensor_d435>

Commit message: raw_height_calculation

File: src/niryo_robot_description/urdf/ned/niryo_ned_gripper1_n_camera.urdf.xacro (robot description, xacro)
@@ -53,6 +53,5 @@
     </link>
     <!-- Mors 1 -->
-    <link
-            name="mors_1">
+    <link name="mors_1">
         <inertial>
             <origin xyz="-0.0049739 0.0067393 -0.023929"
@@ -153,7 +152,11 @@
     <gazebo reference="mors_1">
         <material>Gazebo/DarkGrey</material>
+        <kp>1000000.0</kp>      <kd>10.0</kd>          <mu1>1.5</mu1>         <mu2>1.5</mu2>         <minDepth>0.001</minDepth>
+        <maxVel>0.01</maxVel>
     </gazebo>
     <gazebo reference="mors_2">
         <material>Gazebo/DarkGrey</material>
+        <kp>1000000.0</kp>      <kd>10.0</kd>          <mu1>1.5</mu1>         <mu2>1.5</mu2>         <minDepth>0.001</minDepth>
+        <maxVel>0.01</maxVel>
     </gazebo>
 </robot>
